Commit message: Lowered racecar.urdf wheel interia for accuracy.

File: gym_driving/resources/racecar/racecar.urdf (robot description, URDF)
Before this commit: robot racecar, 13 links, 12 joints
Links:
- link left_front_wheel: mass 0.34055 -> 0.07
- link left_rear_wheel: mass 0.34055 -> 0.07
- link right_front_wheel: mass 0.34055 -> 0.07
- link right_rear_wheel: mass 0.34055 -> 0.07
Joints:
- joint left_front_wheel_joint: limit effort=10 velocity=100 -> effort=10 velocity=200
- joint left_rear_wheel_joint: limit effort=10 velocity=100 -> effort=10 velocity=200
- joint right_front_wheel_joint: limit effort=10 velocity=100 -> effort=10 velocity=200
- joint right_rear_wheel_joint: limit effort=10 velocity=100 -> effort=10 velocity=200

Commit message: Simplified car acceleration. Added breaking, finished steering.

File: gym_driving/resources/racecar/racecar.urdf (robot description, URDF)
Before this commit: robot racecar, 13 links, 12 joints
Links:
- link chassis_inertia: mass 4.0 -> 2.0

Commit message: Added racecar.urdf bounding box.

File: gym_driving/resources/racecar/racecar.urdf (robot description, URDF)
Before this commit: robot racecar, 13 links, 12 joints
Links:
- link chassis: geometry collision box size=0.3 0.5 0.1; visual mesh filename=meshes/chassis.STL
