Commit message: Moving cube, frame skip done checks fixed.

File: gym_driving/resources/cube/cube1.urdf (robot description, URDF)
Before this commit: robot cube1, 1 links, 0 joints
Links:
- link baseLink: mass 1.0 -> 0.1

File: gym_driving/resources/cube/cube2.urdf (robot description, URDF)
Before this commit: robot cube, 1 links, 0 joints
Links:
- link baseLink: mass 1.0 -> 0.1

File: gym_driving/resources/cube/cube3.urdf (robot description, URDF)
Before this commit: robot cube, 1 links, 0 joints
Links:
- link baseLink: mass 1.0 -> .1

File: gym_driving/resources/cube/cube4.urdf (robot description, URDF)
Before this commit: robot cube, 1 links, 0 joints
Links:
- link baseLink: mass 1.0 -> 0.1

File: gym_driving/resources/cube/cube5.urdf (robot description, URDF)
Before this commit: robot cube, 1 links, 0 joints
Links:
- link baseLink: mass 1.0 -> 0.1

Commit message: Changed time step of physics simulation

File: gym_driving/resources/cube/cube1.urdf (robot description, URDF)
Before this commit: robot cube1, 1 links, 0 joints
Links:
- link baseLink: mass 0.1 -> 5

File: gym_driving/resources/cube/cube2.urdf (robot description, URDF)
Before this commit: robot cube, 1 links, 0 joints
Links:
- link baseLink: mass 0.1 -> 5

File: gym_driving/resources/cube/cube3.urdf (robot description, URDF)
Before this commit: robot cube, 1 links, 0 joints
Links:
- link baseLink: mass .1 -> 5

File: gym_driving/resources/cube/cube4.urdf (robot description, URDF)
Before this commit: robot cube, 1 links, 0 joints
Links:
- link baseLink: mass 0.1 -> 5

File: gym_driving/resources/cube/cube5.urdf (robot description, URDF)
Before this commit: robot cube, 1 links, 0 joints
Links:
- link baseLink: mass 0.1 -> 5
